File: Electrical/DartBoardV1/dartBoardV1.sch (EAGLE design)
At the start: 19 parts, among them U1 STM32F407VET6, U2 LSM6DS3DOT_INDICATION

Commit message: New schematic
Parts:
- removed U$2: OV7670, _HenrySilva:OV7670
- removed U$3, U$4: SM03B-GHS-TB, _HenrySilva:SM03B-GHS-TB
- removed U1: STM32F407VET6, _HenrySilva:STM32F407VET6
- added C11: 100nF, rcl:C-USC0603
- added C12, C13, C14, C15: 22pF, rcl:C-USC0603
- added C27, C28, C29, C30: 0.1uF, rcl:C-USC0603
- added C31: 10uF, rcl:C-USC0603
- added C32: 22uF, rcl:C-USC0603
- added JP1: (no value), adafruit:PINHD-2X20
- added R10, R11: 10k, rcl:R-US_R0603
- added S1: KSR223GLFG, _HenrySilva:KSR223GLFG
- added U$8: 2.2uH/NRH2412T2R2MNGH, HenrySilva:MDKK1616T2R2MM
- added U10, U8: Value, _HenrySilva:DRV8835DSSR
- added U11: (no value), microbuilder:VREG_SOT23-5
- added U3: STM32F405RGT6, _HenrySilva:STM32F405RGT6
- added Y1: 12mhz, microbuilder:CRYSTAL2.5X2.0MM
- C1, C3, C5: value 100uF -> 10uF
- C2: value 100uF -> 0.1uF
- C4: value 100uF -> 100nF
- C6: value 10uF -> 0.1uF
- C8: value 1uF -> 100nF
- R1: value 4.7k -> 10k
- R2: value 4.7k -> 100K
- U$1: value SM02B-GHS-TB -> NX3215SA-32.768K-STD-MUA-8; device _HenrySilva:SM02B-GHS-TB -> _HenrySilva:NX3215SA-32.768K-STD-MUA-8
Connections:
- removed net +5V: U$3.2, U$4.2
- removed net PA4: U$2.HREF, U1A.PA4
- removed net PA6: U$2.PCLK, U1A.PA6
- removed net PA8: U$2.XCLK, U1A.PA8
- removed net PB6: U$2.D5, U1A.PB6
- removed net PB7: U$2.VSYNC, U1A.PB7
- removed net PB8: U$2.D6, U1A.PB8
- removed net PB9: U$2.D7, U1A.PB9
- removed net PC11: U$2.D4, U1A.PC11
- removed net PC4: U$2.PWDN
- removed net PC5: U$2.RST, U1A.PC5
- removed net PC6: U$2.D0, U1A.PC6
- removed net PC7: U$2.D1, U1A.PC7
- removed net PC8: U$2.D2, U1A.PC8
- removed net PC9: U$2.D3, U1A.PC9
- new net A1+: U8.AOUT1
- new net A1-: U8.AOUT2
- new net A2+: U8.BOUT1
- new net A2-: U8.BOUT2
- new net A3+: U10.AOUT1
- new net A3-: U10.AOUT2
- new net A4+: U10.BOUT1
- new net A4-: U10.BOUT2
- new net N$17: R2.2, U11.EN
- new net N$18: U$8.1, U11.OUT
- new net N$2: C12.1, U$1.1, U3.PC15/OSC32_OUT
- new net N$3: C1.2, C11.2, C2.2, C4.2, C7.2, C8.2
- new net N$4: C13.1, U$1.2, U3.PC14/OSC32_IN
- new net N$5: C5.1, U3.VCAP_1
- new net N$6: C3.1, U3.VCAP_2
- new net N$7: R1.2, U3.BOOT0
- new net N$8: C14.1, U3.PH1/OSC_OUT, Y1.1
- new net N$9: C15.1, U3.PH0/OSC_IN, Y1.2
- new net P1: U8.AIN1_APHASE
- new net P2: U8.BIN1_BPHASE
- new net P3: U10.AIN1_APHASE
- new net P4: U10.BIN1_BPHASE
- new net PHASE1: U3.PC6
- new net PHASE2: U3.PC7
- new net PHASE3: U3.PC8
- new net PHASE4: U3.PC9
- new net PWM3: U10.AIN2_AENBL, U3.PA10
- new net PWM4: U10.BIN2_BENBL, U3.PA11
- new net RESET: C6.1, S1.1, U3.NRST
- new net RX: JP1.8, U3.PB7
- new net TX: JP1.10, U3.PB6
- net +3V3: now also C11.1, C28.1, C30.1, C32.1, JP1.1, R10.2, R11.2, U$8.2, U10.MODE, U10.VCC, U11.P4, U3.VBAT, U3.VDD, U3.VDDA, U8.MODE, U8.VCC; no longer C3.1, C5.1, C6.1, R1.2, R2.2, U$2.VCC, U1C.VDDA, U1C.VDD_1, U1C.VDD_2, U1C.VDD_3, U1C.VDD_4, U1C.VDD_5, U1C.VREF+
- net GND: now also C12.2, C13.2, C14.2, C15.2, C27.2, C28.2, C29.2, C30.2, C31.2, C32.2, JP1.6, R1.1, S1.2, U10.GND, U10.GND_2, U11.GND, U3.PB2/BOOT1, U3.VSS, U3.VSSA, U8.GND, U8.GND_2; no longer C1.2, C2.2, C4.2, C7.2, C8.2, U$1.2, U$2.GND, U$3.1, U$4.1, U1C.VREF-, U1C.VSSA, U1C.VSS_1, U1C.VSS_2, U1C.VSS_3, U1C.VSS_4, U1C.VSS_5
- net PWM1: now also U3.PA8, U8.AIN2_AENBL; no longer U$3.3, U1B.PE7
- net PWM2: now also U3.PA9, U8.BIN2_BENBL; no longer U$4.3, U1B.PE8
- net SCL: now also R10.1, U3.PB8; no longer R2.1, U$2.SCL, U1A.PB10
- net SDA: now also R11.1, U3.PB9; no longer R1.1, U$2.SD, U1A.PB11
- net VCC: now also C27.1, C29.1, C31.1, R2.1, U10.VM, U11.IN, U8.VM; no longer U$1.1
Other:
- note added: "Buck 3.7v -> 3.3v"
- note added: "DRV8835 (Motor Driver)"
- note added: "Does uart need pullup or pulldown?"
- note added: "To Do: - Connect Pi to 3.3v power - Convert battery power to 3.3v - Make power pins for Dart Trigger Device - Find connectors for wires"
- note removed: "Battery"
- note removed: "Camera"
- note removed: "For VDD 1-5"
- note removed: "For VDDA"
- note removed: "Servo 1"
- note removed: "Servo 2"
- moved on the sheet: C1, C10, C2, C3, C4, C5, C6, C7, C8, C9, R1, R2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
